File: schematics/TTL logic level converter/schematic.sch (EAGLE design)
At the start: 5 parts

Commit message: TTL logic level converter prehodenie 5V a 3V3
Connections:
- net 3V3: now also JP1.1; no longer JP1.2
- net 5V: now also JP1.2; no longer JP1.1
Changed lines of the file:
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@@
 <net name="5V" class="0">
-<segment>
-<pinref part="JP1" gate="A" pin="1"/>
-<wire x1="25.4" y1="119.38" x2="17.78" y2="119.38" width="0.1524" layer="91"/>
-<label x="30.48" y="119.38" size="1.778" layer="95"/>
-<label x="30.48" y="119.38" size="1.778" layer="95"/>
-</segment>
 <segment>
 <pinref part="R1" gate="G$1" pin="1"/>
@@
 <label x="25.4" y="78.74" size="1.778" layer="95"/>
 </segment>
+<segment>
+<pinref part="JP1" gate="A" pin="2"/>
+<wire x1="17.78" y1="116.84" x2="25.4" y2="116.84" width="0.1524" layer="91"/>
+<label x="30.48" y="116.84" size="1.778" layer="95"/>
+</segment>
 </net>
 <net name="3V3" class="0">
-<segment>
-<pinref part="JP1" gate="A" pin="2"/>
-<wire x1="25.4" y1="116.84" x2="17.78" y2="116.84" width="0.1524" layer="91"/>
-<label x="30.48" y="116.84" size="1.778" layer="95"/>
-</segment>
 <segment>
 <pinref part="R2" gate="G$1" pin="1"/>
@@
 <label x="25.4" y="93.98" size="1.778" layer="95"/>
 </segment>
+<segment>
+<pinref part="JP1" gate="A" pin="1"/>
+<wire x1="17.78" y1="119.38" x2="25.4" y2="119.38" width="0.1524" layer="91"/>
+<label x="30.48" y="119.38" size="1.778" layer="95"/>
+</segment>
 </net>
